File: damn_simple_arduino/damn_simple_arduino.sch (KiCad schematic (older format))
At the start: 27 parts, among them IC1 ATMEGA328P-P, P1 USB_B, P2 CONN_01X08, P3 CONN_01X10, P4 CONN_01X06, P5 CONN_01X08, P6 CONN_02X03, U1 FT231XS, Y1 Crystal

Commit message: Updating design to AC couple the reset line to DTR, after bring-up tests.
Connections:
- net Earth: no longer C10.2
- net MCU_RST: no longer U1.1 (~DTR)
- new net: C10.2, U1.1 (~DTR)
Changed lines of the file:
@@
 	1    0    0    -1
 $EndComp
-Text Label 4600 3450 0    60   ~ 0
+Text Label 5250 3450 0    60   ~ 0
 MCU_RST
 Text Label 4600 3050 0    60   ~ 0
@@
 $EndComp
 $Comp
-L Earth #PWR01
+L Earth #PWR13
 U 1 1 5837F21A
 P 10950 4150
-F 0 "#PWR01" H 10950 3900 50  0001 C CNN
+F 0 "#PWR13" H 10950 3900 50  0001 C CNN
 F 1 "Earth" H 10950 4000 50  0001 C CNN
 F 2 "" H 10950 4150 50  0000 C CNN
@@
 MCU_TX
 $Comp
-L Earth #PWR02
+L Earth #PWR9
 U 1 1 5837F7CD
 P 6150 4900
-F 0 "#PWR02" H 6150 4650 50  0001 C CNN
+F 0 "#PWR9" H 6150 4650 50  0001 C CNN
 F 1 "Earth" H 6150 4750 50  0001 C CNN
 F 2 "" H 6150 4900 50  0000 C CNN
@@
 $EndComp
 $Comp
-L Earth #PWR03
+L Earth #PWR6
 U 1 1 5837F8CA
 P 3750 4650
-F 0 "#PWR03" H 3750 4400 50  0001 C CNN
+F 0 "#PWR6" H 3750 4400 50  0001 C CNN
 F 1 "Earth" H 3750 4500 50  0001 C CNN
 F 2 "" H 3750 4650 50  0000 C CNN
@@
 	4450 3150 4600 3150
 Wire Wire Line
-	4450 3450 4600 3450
+	4450 3450 4750 3450
 Wire Wire Line
 	3650 4550 3850 4550
@@
 Connection ~ 3750 4550
 $Comp
-L Earth #PWR04
+L Earth #PWR2
 U 1 1 5837FA24
 P 1750 1850
-F 0 "#PWR04" H 1750 1600 50  0001 C CNN
+F 0 "#PWR2" H 1750 1600 50  0001 C CNN
 F 1 "Earth" H 1750 1700 50  0001 C CNN
 F 2 "" H 1750 1850 50  0000 C CNN
@@
 MCU_5V
 $Comp
-L Earth #PWR05
+L Earth #PWR11
 U 1 1 58380334
 P 7950 1800
-F 0 "#PWR05" H 7950 1550 50  0001 C CNN
+F 0 "#PWR11" H 7950 1550 50  0001 C CNN
 F 1 "Earth" H 7950 1650 50  0001 C CNN
 F 2 "" H 7950 1800 50  0000 C CNN
@@
 	9100 3950 9100 3850
 Connection ~ 9100 3950
-Wire Wire Line
-	9250 4000 9250 3950
-Connection ~ 9250 3950
-$Comp
-L Earth #PWR06
-U 1 1 58380CD9
-P 9250 4350
-F 0 "#PWR06" H 9250 4100 50  0001 C CNN
-F 1 "Earth" H 9250 4200 50  0001 C CNN
-F 2 "" H 9250 4350 50  0000 C CNN
-F 3 "" H 9250 4350 50  0000 C CNN
-	1    9250 4350
-	1    0    0    -1
-$EndComp
-Wire Wire Line
-	9250 4350 9250 4300
 Text Label 9100 3500 0    60   ~ 0
 MCU_5V
@@
 	2450 2000 3700 2000
 $Comp
-L Earth #PWR07
+L Earth #PWR5
 U 1 1 58381037
 P 3050 2050
-F 0 "#PWR07" H 3050 1800 50  0001 C CNN
+F 0 "#PWR5" H 3050 1800 50  0001 C CNN
 F 1 "Earth" H 3050 1900 50  0001 C CNN
 F 2 "" H 3050 2050 50  0000 C CNN
@@
 	2000 3050 2450 3050
 $Comp
-L Earth #PWR08
+L Earth #PWR3
 U 1 1 5838156F
 P 2200 3150
-F 0 "#PWR08" H 2200 2900 50  0001 C CNN
+F 0 "#PWR3" H 2200 2900 50  0001 C CNN
 F 1 "Earth" H 2200 3000 50  0001 C CNN
 F 2 "" H 2200 3150 50  0000 C CNN
@@
 NoConn ~ 2850 6900
 $Comp
-L Earth #PWR09
+L Earth #PWR4
 U 1 1 583874F7
 P 2500 7100
-F 0 "#PWR09" H 2500 6850 50  0001 C CNN
+F 0 "#PWR4" H 2500 6850 50  0001 C CNN
 F 1 "Earth" H 2500 6950 50  0001 C CNN
 F 2 "" H 2500 7100 50  0000 C CNN
@@
 NoConn ~ 5250 6200
 $Comp
-L Earth #PWR010
+L Earth #PWR7
 U 1 1 58388124
 P 5000 7200
-F 0 "#PWR010" H 5000 6950 50  0001 C CNN
+F 0 "#PWR7" H 5000 6950 50  0001 C CNN
 F 1 "Earth" H 5000 7050 50  0001 C CNN
 F 2 "" H 5000 7200 50  0000 C CNN
@@
 $EndComp
 $Comp
-L C C10
-U 1 1 58389081
-P 9250 4150
-F 0 "C10" H 9275 4250 50  0000 L CNN
-F 1 "0.1 uF" H 9275 4050 50  0000 L CNN
-F 2 "Capacitors_SMD:C_0603_HandSoldering" H 9288 4000 50  0001 C CNN
-F 3 "" H 9250 4150 50  0000 C CNN
-F 4 "GRM188R71E104KA01D" H 9250 4150 60  0001 C CNN "manf#"
-	1    9250 4150
-	1    0    0    -1
-$EndComp
-$Comp
 L C C9
 U 1 1 58389399
@@
 $EndComp
 $Comp
-L Earth #PWR011
+L Earth #PWR10
 U 1 1 583894D6
 P 6250 3500
-F 0 "#PWR011" H 6250 3250 50  0001 C CNN
+F 0 "#PWR10" H 6250 3250 50  0001 C CNN
 F 1 "Earth" H 6250 3350 50  0001 C CNN
 F 2 "" H 6250 3500 50  0000 C CNN
@@
 	10000 3750 10350 3750
 $Comp
-L Earth #PWR012
+L Earth #PWR12
 U 1 1 58389C26
 P 10200 4000
-F 0 "#PWR012" H 10200 3750 50  0001 C CNN
+F 0 "#PWR12" H 10200 3750 50  0001 C CNN
 F 1 "Earth" H 10200 3850 50  0001 C CNN
 F 2 "" H 10200 4000 50  0000 C CNN
@@
 	5650 2800 6000 2800
 $Comp
-L Earth #PWR013
+L Earth #PWR8
 U 1 1 5838A4B6
 P 5850 2850
-F 0 "#PWR013" H 5850 2600 50  0001 C CNN
+F 0 "#PWR8" H 5850 2600 50  0001 C CNN
 F 1 "Earth" H 5850 2700 50  0001 C CNN
 F 2 "" H 5850 2850 50  0000 C CNN
@@
 	700  3550 1600 3550
 $Comp
-L Earth #PWR014
+L Earth #PWR1
 U 1 1 5838C53A
 P 1250 4450
-F 0 "#PWR014" H 1250 4200 50  0001 C CNN
+F 0 "#PWR1" H 1250 4200 50  0001 C CNN
 F 1 "Earth" H 1250 4300 50  0001 C CNN
 F 2 "" H 1250 4450 50  0000 C CNN
@@
 Connection ~ 1250 4300
 $Comp
-L PWR_FLAG #FLG015
+L PWR_FLAG #FLG1
 U 1 1 5838D551
 P 5900 2350
-F 0 "#FLG015" H 5900 2445 50  0001 C CNN
+F 0 "#FLG1" H 5900 2445 50  0001 C CNN
 F 1 "PWR_FLAG" H 5900 2530 50  0000 C CNN
 F 2 "" H 5900 2350 50  0000 C CNN
@@
 Connection ~ 5900 2500
 $Comp
-L PWR_FLAG #FLG016
+L PWR_FLAG #FLG2
 U 1 1 5838D97A
 P 8700 1550
-F 0 "#FLG016" H 8700 1645 50  0001 C CNN
+F 0 "#FLG2" H 8700 1645 50  0001 C CNN
 F 1 "PWR_FLAG" H 8700 1730 50  0000 C CNN
 F 2 "" H 8700 1550 50  0000 C CNN
@@
 Connection ~ 5650 2500
 Connection ~ 6000 2500
+$Comp
+L C C10
+U 1 1 5841729D
+P 4900 3450
+F 0 "C10" H 4925 3550 50  0000 L CNN
+F 1 "0.1 uF" H 4925 3350 50  0000 L CNN
+F 2 "Capacitors_SMD:C_0603_HandSoldering" H 4938 3300 50  0001 C CNN
+F 3 "" H 4900 3450 50  0000 C CNN
+F 4 "GRM188R71E104KA01D" H 4900 3450 60  0001 C CNN "manf#"
+	1    4900 3450
+	0    1    1    0
+$EndComp
+Wire Wire Line
+	5050 3450 5250 3450
 $EndSCHEMATC

Commit message: Updating layout with keepout zone for crystal. Also adding BOM.
Other:
- note added: "FTDI Serial-USB Converter"
- note added: "I/O Connectors"
- note added: "ICSP Connector"
- note added: "USB Connector"
- moved on the sheet: C10, P2, P3, P4, P5
