File: arduino++/arduino++.kicad_pcb (KiCad board)
At the start: 4 copper layers, 50.5 x 66 mm, 81 parts, among them IC1 ATMEGA328PB-A, P1 CONN_01X18, P2 CONN_01X03, P3 USB_OTG, P4 CONN_01X03, P5 CONN_01X21, P6 CONN_01X03, P7 CONN_01X03, P8 CONN_02X03, Q1 Q_NMOS_DGS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

Commit message: Updating to latest rev as ordered on OSHPark.
Parts:
- removed ?: Symbol_OSHW-Logo_SilkScreen, Symbols:Symbol_OSHW-Logo_SilkScreen
- added C30: 15 uF, Capacitors_SMD:C_0805_HandSoldering, F.Cu at (136.7, 35.0)
- added D5: LED, LEDs:LED-0603, F.Cu at (116.2, 70.8)
- added R16: 30, Resistors_SMD:R_0402, F.Cu at (119.2, 70.8)
- U2: value NCP551SN33T1G -> TAR5SB33; footprint Housings_SOT-23_SOT-143_TSOT-6:SOT-23-5 -> housings_sot_custom:SC-74A_SOT23-5
- moved C12 6.62 mm to (134.3, 43.1), turned to 270 degrees
- moved C13 2.19 mm to (140.3, 38.2)
- moved U2 1.15 mm to (137.7, 40.7)
Connections:
- C13 pad 1: +3V3 -> Net-(C13-Pad1)
- P3 pad 4: Net-(P3-Pad4) -> (no net)
- U1 pad 10: Net-(U1-Pad10) -> (no net)
- U1 pad 17: Net-(U1-Pad17) -> (no net)
- U1 pad 18: Net-(U1-Pad18) -> (no net)
- U1 pad 19: Net-(U1-Pad19) -> (no net)
- U1 pad 2: Net-(U1-Pad2) -> (no net)
- U1 pad 5: Net-(U1-Pad5) -> (no net)
- U1 pad 7: Net-(U1-Pad7) -> (no net)
- U1 pad 8: Net-(U1-Pad8) -> (no net)
- U1 pad 9: Net-(U1-Pad9) -> (no net)
- U2 pad 3: Net-(U2-Pad3) -> Net-(C12-Pad1)
- U2 pad 4: Net-(U2-Pad4) -> Net-(C13-Pad1)
- U7 pad 11: Net-(U7-Pad11) -> (no net)
Routing:
- net /SPICLK: track 70.5 -> 76.4 mm, vias 1 -> 3
- net Net-(C12-Pad1): track 15.3 -> 19.1 mm
- net Earth: track 92.2 -> 95.5 mm, vias 54 -> 56
- net +3V3: track 98.2 -> 101.6 mm, vias 8 -> 9
- net Net-(C13-Pad1): track 0.00 -> 1.94 mm
- net Net-(D5-Pad2): track 0.00 -> 1.80 mm
Other:
- board text added: "PCB: POLYBOTS002-001 PCBA: POLYBOTS002-101"
- board text added: "RoboBoard Dev-0.1 DE: Abhimanyu Ghosh NYU PolyBOTS"
- board text removed: "RoboBoard Dev-0.1 RE: Abhimanyu Ghosh NYU PolyBOTS"
