File: stm32_interface_board/MotorDriver.sch (KiCad schematic (older format))
At the start: 9 parts, among them U1 A3909

Commit message: Adding latest STM32 Interface board files.
Parts:
- removed C3, C4: 22 uF, Capacitors_SMD:C_1206_HandSoldering, symbol C
Changed lines of the file:
@@
 LIBS:PowerManagement
 LIBS:ftdi
+LIBS:mechanical
 LIBS:stm32_interface_board-cache
 EELAYER 25 0
@@
 $EndComp
 $Comp
-L Earth #PWR29
+L Earth #PWR031
 U 1 1 58B85868
 P 4550 4650
-F 0 "#PWR29" H 4550 4400 50  0001 C CNN
+F 0 "#PWR031" H 4550 4400 50  0001 C CNN
 F 1 "Earth" H 4550 4500 50  0001 C CNN
 F 2 "" H 4550 4650 50  0000 C CNN
@@
 $EndComp
 $Comp
-L Earth #PWR31
+L Earth #PWR032
 U 1 1 58B85952
 P 7300 4600
-F 0 "#PWR31" H 7300 4350 50  0001 C CNN
+F 0 "#PWR032" H 7300 4350 50  0001 C CNN
 F 1 "Earth" H 7300 4450 50  0001 C CNN
 F 2 "" H 7300 4600 50  0000 C CNN
@@
 	7300 3700 7050 3700
 Connection ~ 7300 3700
-Text HLabel 8450 3000 2    60   Output ~ 0
+Text HLabel 8450 3500 2    60   Output ~ 0
 M1P
 Text HLabel 8450 3600 2    60   Output ~ 0
@@
 Text HLabel 8450 3800 2    60   Output ~ 0
 M2P
-Text HLabel 8450 4400 2    60   Output ~ 0
+Text HLabel 8450 3900 2    60   Output ~ 0
 M2N
 $Comp
@@
 $EndComp
 $Comp
-L +BATT #PWR28
+L +BATT #PWR033
 U 1 1 58B85D2F
 P 3500 2600
-F 0 "#PWR28" H 3500 2450 50  0001 C CNN
+F 0 "#PWR033" H 3500 2450 50  0001 C CNN
 F 1 "+BATT" H 3500 2740 50  0000 C CNN
 F 2 "" H 3500 2600 50  0000 C CNN
@@
 	7050 3600 8450 3600
 Wire Wire Line
-	7050 3500 7550 3500
-Wire Wire Line
-	7550 3500 7550 3000
-Wire Wire Line
-	7550 3000 8450 3000
+	7050 3500 8450 3500
 Wire Wire Line
 	7050 3800 8450 3800
 Wire Wire Line
-	7050 3900 7550 3900
-Wire Wire Line
-	7550 3900 7550 4400
-Wire Wire Line
-	7550 4400 8450 4400
+	7050 3900 8450 3900
 $Comp
 L C C2
@@
 	1    0    0    -1
 $EndComp
-$Comp
-L C C3
-U 1 1 58B8C34D
-P 8050 3250
-F 0 "C3" H 8075 3350 50  0000 L CNN
-F 1 "22 uF" H 8075 3150 50  0000 L CNN
-F 2 "Capacitors_SMD:C_1206_HandSoldering" H 8088 3100 50  0001 C CNN
-F 3 "" H 8050 3250 50  0000 C CNN
-F 4 "TMK316BBJ226ML-T" H 8050 3250 60  0001 C CNN "manf#"
-	1    8050 3250
-	1    0    0    -1
-$EndComp
-$Comp
-L C C4
-U 1 1 58B8C407
-P 8050 4050
-F 0 "C4" H 8075 4150 50  0000 L CNN
-F 1 "22 uF" H 8075 3950 50  0000 L CNN
-F 2 "Capacitors_SMD:C_1206_HandSoldering" H 8088 3900 50  0001 C CNN
-F 3 "" H 8050 4050 50  0000 C CNN
-F 4 "TMK316BBJ226ML-T" H 8050 4050 60  0001 C CNN "manf#"
-	1    8050 4050
-	1    0    0    -1
-$EndComp
-Wire Wire Line
-	8050 4200 8050 4400
-Connection ~ 8050 4400
-Wire Wire Line
-	8050 3900 8050 3800
-Connection ~ 8050 3800
-Wire Wire Line
-	8050 3600 8050 3400
-Connection ~ 8050 3600
-Wire Wire Line
-	8050 3100 8050 3000
-Connection ~ 8050 3000
 Connection ~ 4400 2600
 Connection ~ 4950 2600
@@
 	4400 2900 4950 2900
 $Comp
-L Earth #PWR30
+L Earth #PWR034
 U 1 1 58B8C6D0
 P 4650 3000
-F 0 "#PWR30" H 4650 2750 50  0001 C CNN
+F 0 "#PWR034" H 4650 2750 50  0001 C CNN
 F 1 "Earth" H 4650 2850 50  0001 C CNN
 F 2 "" H 4650 3000 50  0000 C CNN
