File: stm32_interface_board/stm32_interface_board.kicad_pcb (KiCad board)
At the start: 2 copper layers, 75 x 87.5 mm, 38 parts, among them P1 USB_OTG, P10 CONN_01X03, P11 CONN_01X02, P2 CONN_02X25, P3 CONN_02X25, P4 CONN_01X04, P5 CONN_01X04, P6 CONN_01X04, P7 CONN_01X02, P8 CONN_01X02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

Commit message: Fixing DRC issues.
Parts:
- moved C13 2.15 mm to (92.6, 106.2)
Routing:
- net +5V: track 184.8 -> 182.8 mm
Other:
- net class Default: via_dia 0.6 -> 0.7
- rule via_min_drill: 0.3 -> 0.4
- rule via_min_size: 0.4 -> 0.7

Commit message: Adding latest STM32 Interface board files.
Parts:
- removed C3, C4: 22 uF, Capacitors_SMD:C_1206_HandSoldering
- removed REF**: Symbol_OSHW-Logo_SilkScreen, Symbols:Symbol_OSHW-Logo_SilkScreen
- added TH1: PTH, mechanical:PTH, F.Cu at (120.0, 60.0)
- added TH2: PTH, mechanical:PTH, F.Cu at (140.0, 60.0)
- added TH3: PTH, mechanical:PTH, F.Cu at (140.0, 80.0)
- moved P9 77.2 mm to (160.3, 105.3)
- moved P10 70.9 mm to (160.3, 94.8)
- moved C12 17.1 mm to (90.0, 107.7), turned to 0 degrees
- moved U3 14.3 mm to (91.3, 104.5), turned to 0 degrees
- moved R4 6.05 mm to (115.2, 84.2), turned to 180 degrees
- moved C13 5.93 mm to (91.0, 111.8)
- moved U1 4.15 mm to (112.5, 116.2)
- moved C1 3.20 mm to (110.5, 106.7)
- moved C2 2.65 mm to (113.4, 109.5)
- moved P7 0.40 mm to (118.7, 122.5)
- moved P8 0.15 mm to (108.5, 122.5)
Connections:
- net /MotorDriver/M1_PWM2 renamed /M1_2
- net /MotorDriver/M2_PWM1 renamed /M2_1
- P2 pad 11: (no net) -> /AIN0
- P2 pad 14: (no net) -> /AIN1
- P2 pad 22: (no net) -> /ECHO2
- P2 pad 5: (no net) -> /TRIG2
- P3 pad 11: /MCU_RX -> (no net)
- P3 pad 14: /MCU_TX -> (no net)
- P3 pad 19: /AIN0 -> (no net)
- P3 pad 20: /AIN1 -> (no net)
- P3 pad 27: /MotorDriver/M1_PWM1 -> (no net)
- P3 pad 28: (no net) -> /M1_1
- P3 pad 30: (no net) -> /M2_2
- P3 pad 32: /MotorDriver/M2_PWM2 -> (no net)
- P3 pad 34: (no net) -> /TRIG1
- P3 pad 40: /ECHO2 -> (no net)
- P3 pad 41: /TRIG1 -> (no net)
- P3 pad 42: /TRIG2 -> (no net)
- P3 pad 43: (no net) -> /MCU_RX
- P3 pad 44: (no net) -> /MCU_TX
- R1 pad 1: /MotorDriver/M2_PWM2 -> /M2_2
- R4 pad 1: /MotorDriver/M1_PWM1 -> /M1_1
- U1 pad 1: /MotorDriver/M1_PWM1 -> /M1_1
- U1 pad 5: /MotorDriver/M2_PWM2 -> /M2_2
Routing:
- net +5V: track 182.8 -> 3.20 mm
- net /TRIG2: track 21.9 -> 128.9 mm, vias 0 -> 2
- net /ECHO2: track 21.7 -> 99.4 mm, vias 0 -> 2
- net /M1_1: track 0.00 -> 63.0 mm
- net /MotorDriver/M2_PWM2: track 61.0 -> 0.00 mm
- net /M2_2: track 0.00 -> 58.1 mm
- net /MotorDriver/M1_PWM1: track 52.8 -> 0.00 mm
- net Earth: track 77.2 -> 48.1 mm, vias 19 -> 22
- net /MCU_TX: track 101.6 -> 88.6 mm, vias 0 -> 1
- net /TRIG1: track 42.7 -> 54.8 mm
- net /MCU_RX: track 77.3 -> 87.1 mm, vias 0 -> 1
- net /M1_2: track 50.8 -> 57.9 mm
- net /MotorDriver/M1P: track 14.1 -> 8.23 mm
- net /MotorDriver/M2N: track 13.6 -> 8.52 mm
- net /MotorDriver/M1N: track 10.7 -> 6.42 mm
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- added copper zone on F.Cu, net +5V
Other:
- board size 75 x 87.5 mm -> 75 x 88 mm
- board text added: "Batt"
- board text added: "Debug-USART1"
- board text added: "M1"
- board text added: "M2"
- board text added: "STM32 Robot Interface Board Abhimanyu Ghosh 2017 Release-0.1"
- board text removed: "STM32 Robot Interface Board Abhimanyu Ghosh 2017"

Commit message: Updating STM Interface board to latest rev.
Parts:
- added TH4: PTH, mechanical:PTH, F.Cu at (109.7, 74.5)
- moved R4 29.3 mm to (119.9, 113.2), turned to 0 degrees
- moved R3 21.7 mm to (115.4, 103.8), turned to 180 degrees
- moved TH1 14.2 mm to (109.7, 50.2)
- moved R1 11.9 mm to (106.7, 98.7)
- moved R2 11.8 mm to (113.7, 98.6)
- moved TH2 9.83 mm to (140.0, 50.2)
- moved P8 7.33 mm to (102.8, 118.0), turned to 90 degrees
- moved TH3 5.52 mm to (140.0, 74.5)
- moved P7 4.72 mm to (119.9, 118.0), turned to 90 degrees
Connections:
- P10 pad 2: +5V -> Earth
- P10 pad 3: Earth -> +5V
- P2 pad 22: /ECHO2 -> /TRIG2
- P2 pad 5: /TRIG2 -> (no net)
- P3 pad 3: (no net) -> /ECHO2
- P9 pad 2: +5V -> Earth
- P9 pad 3: Earth -> +5V
Routing:
- net /ECHO2: track 99.4 -> 71.4 mm, vias 2 -> 0
- net /TRIG2: track 128.9 -> 102.7 mm
- net /M1_2: track 57.9 -> 48.4 mm
- net /MotorDriver/M1N: track 6.42 -> 12.5 mm
- net /MotorDriver/M2P: track 6.60 -> 11.9 mm
- net /M1_1: track 63.0 -> 59.1 mm
- net /M2_2: track 58.1 -> 61.4 mm, vias 0 -> 2
- net /M2_1: track 58.8 -> 61.1 mm, vias 0 -> 2
- net /MotorDriver/M2N: track 8.52 -> 6.34 mm
- net /MotorDriver/M1P: track 8.23 -> 6.68 mm
- net /ECHO1: track 42.1 -> 43.2 mm
- net +BATT: track 57.2 -> 56.3 mm, vias 1 -> 0
